File: hardware/am24_shield.kicad_sch (KiCad schematic)
At the start: 88 parts, among them J5 +5V -> E5V (CN7-6), J6 TCXO -> OSC_IN (PF0), U1 NXE1S0505MC, X1 IN 4-20 mA, X2 24V DC, X3 OUT 1: OC/PP/0V, X4 OUT 2: OC/PP/0V

Commit message: 0.001 % pulse output: chopped ADC, NTC compensation, GPS clock
- firmware 0.2.0: AIN0/AIN1 swapped pairs cancel ADC offset; NTC on
  AIN6 with per-unit tc_ppm; up to 11 calibration points in double;
  WIN START / WIN? averaging window; GPS PPS on D6 (PB10, TIM2_CH3)
  measures the TCXO and latches the exact pulse total on each edge;
  frequency output moved to TIM5 (same pin PA0); clock correction now
  also applies to the pulse integrator (was frequency output only);
  settings format v2
- hardware: RK1/R9/C33 NTC divider from VREF, J7 GPS connector + R10
  to D6; BOM updated
- tools/am24.py: multimeter over VISA (SCPI or 3458A) or manual entry,
  cal (9 points), verify (+-10 ppm), tempco, pulses (GPS time), gps
- docs: 0.001 % error budget, BOM, availability, calibration procedure

Co-Authored-By: Claude Opus 5.5 <noreply@anthropic.com>
Parts:
- added C33: 100n, Capacitor_SMD:C_0805_2012Metric, symbol Device:C
- added J7: GPS PPS, Connector_PinHeader_2.54mm:PinHeader_1x04_P2.54mm_Vertical, symbol Connector_Generic:Conn_01x04
- added R10: 100R, Resistor_SMD:R_0805_2012Metric, symbol Device:R
- added R9: 10k 0.1%, Resistor_SMD:R_0805_2012Metric, symbol Device:R
- added RK1: 10k B3380, Resistor_SMD:R_0603_1608Metric, symbol Device:Thermistor_NTC
Connections:
- net +3V3: now also J7.2 (Pin_2)
- net +5V: now also J7.1 (Pin_1)
- net AGND: now also C33.2, RK1.2
- net GND: now also J7.3 (Pin_3)
- net at C16.1, DA1.6 (VOUT_S), DA1.7 (VOUT_F)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: now also R9.1
- net NTC: now reaches DD1.16 (AIN6/REFIN2+)
- net NTC: now also C33.1, R9.2, RK1.1
- net at XS4.7 (Pin_7): now also R10.2
- new net: J7.4 (Pin_4), R10.1
- no-connect marks 32 -> 30
Other:
- note added: "J7: модуль GPS с выходом PPS. 1 +5V, 2 +3V3, 3 GND, 4 PPS -> D6 (PB10)"
- note added: "RK1 вплотную к DA1 и R2, всё под крышкой"

Commit message: Footprint for F1/F2: Bourns MF-R radial PTC
- hardware/am24.pretty: Fuse_Bourns_MF-R_8.0x3.1mm_P5.10mm, drawn from
  the Bourns MF-R datasheet (pitch 5.1 mm, leads ~1.8 mm apart across
  the 3.1 mm body, 0.8 mm drill for 0.405-0.51 mm leads)
- hardware/fp-lib-table: project library AM24
- F1 (MF-R005-0) and F2 (MF-R050) use it; BOM and README updated

Co-Authored-By: Claude Opus 5.5 <noreply@anthropic.com>
Parts:
- F1, F2: footprint (none) -> AM24:Fuse_Bourns_MF-R_8.0x3.1mm_P5.10mm

Commit message: PCB: 100 x 90 mm shield, 4-layer and 2-layer variants
- tools/gen_pcb.py: outline with slots over Morpho CN7 pins 29/6,
  placement in the Nucleo-64 frame (Arduino headers on the bottom,
  through-hole parts only off the Nucleo), 4 mm copper-free isolation
  barrier crossed only by ISO7741 and NXE1, net classes, hand-routed
  Kelvin lines from the shunt, In1 AGND/GND plane on 4 layers
- tools/route_pcb.py: Freerouting (headless), ground pours, drain
  copper under the OC DPAKs, stitching vias, dead-end cleanup
- tools/export_fab.py: Gerber, drill and position files per board
- hardware: both boards, fab zips, renders, top assembly drawing;
  J5/J6 changed to SMD pin headers
- DRC: no unconnected nets, clearance violations or shorts

Co-Authored-By: Claude Opus 5.5 <noreply@anthropic.com>
Parts:
- J5, J6: footprint Connector_PinHeader_2.54mm:PinHeader_1x02_P2.54mm_Vertical -> Connector_PinHeader_2.54mm:PinHeader_1x02_P2.54mm_Vertical_SMD_Pin1Left
